File: mf.kicad_pcb (KiCad board)
At the start: 2 copper layers, 363 x 166.2 mm, 121 parts, among them U1 Sparkfun_Pro_Micro, U10 74HC165, U11 DM13a, U14 74HC165, U16 74HC165, U17 74HC165, U19 74HC165, U5 74HC165, U6 74HC165, U7 Sparkfun_Pro_Micro, U8 74HC165, U9 DM13a

Commit message: Begin PCB routing + change in schematic
Parts:
- removed C4: Capacitor_NP, Capacitor_THT:C_Disc_D3.0mm_W2.0mm_P2.50mm
- removed R25, R26, R27, R28, R29, R30, R31, R32, R67, R68, R69, R70, R71, R72, R73, R74, R75, R76, R77, R78, R79, R80, R81, R82: Resistor, Resistor_THT:R_Axial_DIN0207_L6.3mm_D2.5mm_P10.16mm_Horizontal
- removed RB6: ~, mf:r_but
- removed U10: 74HC165, Package_DIP:DIP-16_W7.62mm_LongPads
- added R1: Resistor, Resistor_THT:R_Axial_DIN0207_L6.3mm_D2.5mm_P10.16mm_Horizontal, B.Cu at (361.8, 183.0)
- added R10: Resistor, Resistor_THT:R_Axial_DIN0207_L6.3mm_D2.5mm_P10.16mm_Horizontal, B.Cu at (167.5, 186.0)
- added R11: Resistor, Resistor_THT:R_Axial_DIN0207_L6.3mm_D2.5mm_P10.16mm_Horizontal, B.Cu at (167.5, 189.0)
- added R12: Resistor, Resistor_THT:R_Axial_DIN0207_L6.3mm_D2.5mm_P10.16mm_Horizontal, B.Cu at (167.5, 192.0)
- added R13: Resistor, Resistor_THT:R_Axial_DIN0207_L6.3mm_D2.5mm_P10.16mm_Horizontal, B.Cu at (205.1, 192.0)
- added R14: Resistor, Resistor_THT:R_Axial_DIN0207_L6.3mm_D2.5mm_P10.16mm_Horizontal, B.Cu at (205.1, 189.0)
- added R15: Resistor, Resistor_THT:R_Axial_DIN0207_L6.3mm_D2.5mm_P10.16mm_Horizontal, B.Cu at (205.1, 186.0)
- added R16: Resistor, Resistor_THT:R_Axial_DIN0207_L6.3mm_D2.5mm_P10.16mm_Horizontal, B.Cu at (205.1, 183.0)
- added R2: Resistor, Resistor_THT:R_Axial_DIN0207_L6.3mm_D2.5mm_P10.16mm_Horizontal, B.Cu at (361.8, 186.0)
- added R3: Resistor, Resistor_THT:R_Axial_DIN0207_L6.3mm_D2.5mm_P10.16mm_Horizontal, B.Cu at (361.8, 189.0)
- added R4: Resistor, Resistor_THT:R_Axial_DIN0207_L6.3mm_D2.5mm_P10.16mm_Horizontal, B.Cu at (361.8, 192.0)
- added R5: Resistor, Resistor_THT:R_Axial_DIN0207_L6.3mm_D2.5mm_P10.16mm_Horizontal, B.Cu at (324.2, 192.0)
- added R6: Resistor, Resistor_THT:R_Axial_DIN0207_L6.3mm_D2.5mm_P10.16mm_Horizontal, B.Cu at (324.2, 189.0)
- added R7: Resistor, Resistor_THT:R_Axial_DIN0207_L6.3mm_D2.5mm_P10.16mm_Horizontal, B.Cu at (324.2, 186.0)
- added R8: Resistor, Resistor_THT:R_Axial_DIN0207_L6.3mm_D2.5mm_P10.16mm_Horizontal, B.Cu at (324.2, 183.0)
- added R9: Resistor, Resistor_THT:R_Axial_DIN0207_L6.3mm_D2.5mm_P10.16mm_Horizontal, B.Cu at (167.5, 183.0)
- added U21: ~, mf:3posswitch, F.Cu at (184.5, 163.0)
- added U22: ~, mf:3posswitch, F.Cu at (199.5, 163.0)
- U7: moved to B.Cu
- moved U1 273.0 mm to (328.7, 125.4), turned to 90 degrees
- moved C9 246.9 mm to (129.0, 196.0)
- moved R37 217.7 mm to (158.0, 182.4), turned to -90 degrees
- moved BC20 189.5 mm to (34.5, 91.0)
- moved BC16 188.3 mm to (58.5, 115.0)
- moved U16 171.2 mm to (114.7, 122.6), turned to 0 degrees
- moved R55 164.9 mm to (75.8, 192.0), turned to 0 degrees
- moved R56 162.7 mm to (75.8, 189.0), turned to 0 degrees
- moved R57 160.6 mm to (75.8, 186.0), turned to 0 degrees
- moved R58 158.7 mm to (75.8, 183.0), turned to 0 degrees
- moved R39 157.6 mm to (219.8, 192.0), turned to 0 degrees
- moved R40 155.4 mm to (219.8, 189.0), turned to 0 degrees
- moved BC17 154.4 mm to (34.5, 115.0)
- moved R41 153.4 mm to (219.8, 186.0), turned to 0 degrees
- moved R42 151.7 mm to (219.8, 183.0), turned to 0 degrees
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- renumbered U19 to U16, U16 to U19
Connections:
- BC1 pad 2: Net-(BC1-C) -> GND
- BC1 pad 5: +5V -> +5VPW
- BC10 pad 2: Net-(BC1-C) -> GND
- BC10 pad 5: +5V -> +5VPW
- BC11 pad 2: Net-(BC1-C) -> GND
- BC11 pad 5: +5V -> +5VPW
- BC12 pad 2: Net-(BC1-C) -> GND
- BC12 pad 5: +5V -> +5VPW
- BC13 pad 2: Net-(BC1-C) -> GND
- BC13 pad 5: +5V -> +5VPW
- BC14 pad 2: Net-(BC1-C) -> GND
- BC14 pad 5: +5V -> +5VPW
- BC15 pad 5: +5V -> +5VPW
- BC16 pad 5: +5V -> +5VPW
- BC17 pad 5: +5V -> +5VPW
- BC18 pad 5: +5V -> +5VPW
- BC19 pad 5: +5V -> +5VPW
- BC2 pad 2: Net-(BC1-C) -> GND
- BC2 pad 5: +5V -> +5VPW
- BC20 pad 5: +5V -> +5VPW
- BC3 pad 2: Net-(BC1-C) -> GND
- BC3 pad 5: +5V -> +5VPW
- BC4 pad 2: Net-(BC1-C) -> GND
- BC4 pad 5: +5V -> +5VPW
- BC5 pad 2: Net-(BC1-C) -> GND
- BC5 pad 5: +5V -> +5VPW
- BC6 pad 2: Net-(BC1-C) -> GND
- BC6 pad 5: +5V -> +5VPW
- BC7 pad 2: Net-(BC1-C) -> GND
- BC7 pad 5: +5V -> +5VPW
- BC8 pad 2: Net-(BC1-C) -> GND
- BC8 pad 5: +5V -> +5VPW
- BC9 pad 2: Net-(BC1-C) -> GND
- BC9 pad 5: +5V -> +5VPW
- C10 pad 2: +5V -> +5VPW
- C9 pad 2: +5V -> +5VPW
- E5 pad 2: Net-(E5-COM) -> GND
- E5 pad 5: Net-(E5-COM) -> GND
- R17 pad 2: Net-(E1-D) -> Net-(BC3-NO)
- R18 pad 2: Net-(E2-D) -> Net-(U8-D1)
- R19 pad 2: Net-(E3-D) -> Net-(U8-D2)
- R20 pad 2: Net-(E4-D) -> Net-(U8-D3)
- R21 pad 2: Net-(U5-D4) -> Net-(E3-D)
- R22 pad 2: Net-(U5-D5) -> Net-(BC5-NO)
- R23 pad 2: Net-(U5-D6) -> Net-(BC4-NO)
- R24 pad 2: Net-(BC15-NO) -> Net-(U8-D7)
- R34 pad 2: Net-(U8-D0) -> Net-(BC6-NO)
- R35 pad 2: Net-(U8-D1) -> Net-(U14-D1)
- R36 pad 2: Net-(U8-D2) -> Net-(E4-D)
- R38 pad 2: Net-(U8-D3) -> Net-(U14-D3)
- R39 pad 2: Net-(U8-D4) -> Net-(U14-D4)
- R40 pad 2: Net-(U8-D5) -> Net-(U14-D5)
- R41 pad 2: Net-(U8-D6) -> Net-(U14-D6)
- R42 pad 2: Net-(U8-D7) -> Net-(U14-D7)
- R43 pad 2: Net-(U10-D0) -> Net-(U12-1)
- R44 pad 2: Net-(U10-D1) -> Net-(U12-2)
- R45 pad 2: Net-(U10-D2) -> Net-(U12-3)
- R46 pad 2: Net-(U10-D3) -> Net-(U12-4)
- R47 pad 2: Net-(U10-D4) -> Net-(U13-6)
- R48 pad 2: Net-(U10-D5) -> Net-(U13-5)
- R49 pad 2: Net-(U10-D6) -> Net-(U13-4)
- R50 pad 2: Net-(U10-D7) -> Net-(U12-5)
- R51 pad 2: Net-(BC7-NO) -> Net-(U17-D0)
- R53 pad 2: Net-(BC9-NO) -> Net-(E5-D)
- R54 pad 2: Net-(BC10-NO) -> Net-(BC7-NO)
- R55 pad 2: Net-(BC11-NO) -> Net-(BC18-NO)
- R56 pad 2: Net-(BC12-NO) -> Net-(BC15-NO)
- R57 pad 2: Net-(BC13-NO) -> Net-(BC12-NO)
- R58 pad 2: Net-(BC14-NO) -> Net-(BC9-NO)
- R59 pad 1: +5V -> Net-(BC10-NO)
- R59 pad 2: Net-(BC1-NO) -> +5V
- R60 pad 1: +5V -> Net-(BC13-NO)
- R60 pad 2: Net-(BC2-NO) -> +5V
- R61 pad 1: +5V -> Net-(BC16-NO)
- R61 pad 2: Net-(BC3-NO) -> +5V
- R62 pad 1: +5V -> Net-(BC19-NO)
- R62 pad 2: Net-(BC4-NO) -> +5V
- R63 pad 2: Net-(BC5-NO) -> Net-(BC20-NO)
- R64 pad 2: Net-(BC6-NO) -> Net-(BC17-NO)
- R65 pad 2: Net-(E5-D) -> Net-(BC14-NO)
- R66 pad 2: Net-(U16-D7) -> Net-(BC11-NO)
- RB4 pad 2: Net-(U5-D4) -> Net-(U14-D1)
- RB5 pad 1: GND -> Net-(U8-D7)
- RB5 pad 2: Net-(U5-D5) -> GND
- U11 pad 15: unconnected-(U11-OUT10-Pad15) -> /Input/LED_BC1
- U11 pad 16: unconnected-(U11-OUT11-Pad16) -> /Input/LED_BC2
- U11 pad 17: unconnected-(U11-OUT12-Pad17) -> /Input/LED_BC3
- U11 pad 18: unconnected-(U11-OUT13-Pad18) -> /Input/LED_BC4
- U11 pad 19: unconnected-(U11-OUT14-Pad19) -> /Input/LED_BC5
- U11 pad 20: unconnected-(U11-OUT15-Pad20) -> /Input/LED_BC6
- U11 pad 24: +5V -> +5VPW
- U11 pad 5: /Input/LED_BC17 -> unconnected-(U11-OUT0-Pad5)
- U11 pad 6: /Input/LED_BC18 -> unconnected-(U11-OUT1-Pad6)
- U11 pad 7: /Input/LED_BC19 -> unconnected-(U11-OUT2-Pad7)
- U11 pad 8: /Input/LED_BC20 -> unconnected-(U11-OUT3-Pad8)
- U14 pad 1: /Input/I_LATCH_L -> Net-(U14-~{PL})
- U14 pad 10: unconnected-(U14-DS-Pad10) -> Net-(U14-DS)
- U14 pad 11: Net-(BC7-NO) -> Net-(BC6-NO)
- U14 pad 12: Net-(BC8-NO) -> Net-(U14-D1)
- U14 pad 13: Net-(BC9-NO) -> Net-(E4-D)
- U14 pad 14: Net-(BC10-NO) -> Net-(U14-D3)
- U14 pad 15: Net-(E5-COM) -> GND
- U14 pad 2: /Input/I_CLK_L -> Net-(U14-CP)
- U14 pad 3: Net-(BC11-NO) -> Net-(U14-D4)
- U14 pad 4: Net-(BC12-NO) -> Net-(U14-D5)
- U14 pad 5: Net-(BC13-NO) -> Net-(U14-D6)
- U14 pad 6: Net-(BC14-NO) -> Net-(U14-D7)
- U14 pad 8: Net-(E5-COM) -> GND
- U15 pad 1: Net-(U16-D7) -> Net-(U6-D4)
- U15 pad 2: Net-(U17-D5) -> Net-(U6-D3)
- U16 pad 1: /Input/I_LATCH_L -> /Input/I_LATCH_R
- U16 pad 10: Net-(U17-Q7) -> Net-(U16-DS)
- U16 pad 11: Net-(U19-D0) -> Net-(U12-5)
- U16 pad 12: Net-(U19-D1) -> Net-(U13-4)
- U16 pad 13: Net-(U12-1) -> Net-(U13-5)
- U16 pad 14: Net-(U12-2) -> Net-(U13-6)
- U16 pad 15: Net-(E5-COM) -> GND
- U16 pad 2: /Input/I_CLK_L -> /Input/I_CLK_R
- U16 pad 3: Net-(U12-3) -> Net-(U12-4)
- U16 pad 4: Net-(U12-4) -> Net-(U12-3)
- U16 pad 5: Net-(U12-5) -> Net-(U12-2)
- U16 pad 6: Net-(U12-6) -> Net-(U12-1)
- U16 pad 8: Net-(E5-COM) -> GND
- U16 pad 9: /Input/I_DATA_L -> Net-(U16-Q7)
- U17 pad 1: /Input/I_LATCH_L -> /Input/I_LATCH_R
- U17 pad 10: Net-(U16-Q7) -> unconnected-(U17-DS-Pad10)
- U17 pad 11: Net-(U13-6) -> Net-(U17-D0)
- U17 pad 12: Net-(U13-5) -> Net-(BC8-NO)
- U17 pad 13: Net-(U13-4) -> Net-(E5-D)
- U17 pad 14: Net-(U13-3) (its old number) -> Net-(BC7-NO)
- U17 pad 15: Net-(E5-COM) -> GND
- U17 pad 2: /Input/I_CLK_L -> /Input/I_CLK_R
- U17 pad 3: Net-(U13-2) (its old number) -> Net-(BC18-NO)
- U17 pad 4: Net-(U17-D5) -> Net-(BC15-NO)
- U17 pad 5: Net-(U17-D6) -> Net-(BC12-NO)
- U17 pad 6: Net-(U17-D7) -> Net-(BC9-NO)
- U17 pad 8: Net-(E5-COM) -> GND
- U18 pad 1: Net-(U17-D7) -> Net-(U6-D2)
- U18 pad 2: Net-(U17-D6) -> Net-(U6-D1)
- U19 pad 1: /Input/I_LATCH_L -> /Input/I_LATCH_R
- U19 pad 10: Net-(U14-Q7) -> Net-(U16-Q7)
- U19 pad 11: Net-(BC1-NO) -> Net-(BC10-NO)
- U19 pad 12: Net-(BC2-NO) -> Net-(BC13-NO)
- U19 pad 13: Net-(BC3-NO) -> Net-(BC16-NO)
- U19 pad 14: Net-(BC4-NO) -> Net-(BC19-NO)
- U19 pad 15: Net-(E5-COM) -> GND
- U19 pad 2: /Input/I_CLK_L -> /Input/I_CLK_R
- U19 pad 3: Net-(BC5-NO) -> Net-(BC20-NO)
- U19 pad 4: Net-(BC6-NO) -> Net-(BC17-NO)
- U19 pad 5: Net-(E5-D) -> Net-(BC14-NO)
- U19 pad 6: Net-(U16-D7) -> Net-(BC11-NO)
- U19 pad 8: Net-(E5-COM) -> GND
- U19 pad 9: Net-(U16-Q7) -> /Input/I_DATA_R
- U2 pad 1: +5V -> +5VPW
- U20 pad 1: Net-(U19-D1) -> Net-(U14-D7)
- U20 pad 2: Net-(U19-D0) -> Net-(U14-D3)
- U4 pad 1: +5V -> +5VPW
- U5 pad 1: /Input/I_LATCH_R -> Net-(U14-~{PL})
- U5 pad 11: Net-(E1-D) -> Net-(BC1-NO)
- U5 pad 12: Net-(E2-D) -> Net-(E1-D)
- U5 pad 13: Net-(E3-D) -> Net-(U5-D2)
- U5 pad 14: Net-(E4-D) -> Net-(U5-D3)
- U5 pad 15: Net-(U10-GND) -> GND
- U5 pad 2: /Input/I_CLK_R -> Net-(U14-CP)
- U5 pad 5: Net-(U5-D6) -> Net-(BC2-NO)
- U5 pad 6: Net-(BC15-NO) -> Net-(E2-D)
- U5 pad 8: Net-(U10-GND) -> GND
- U6 pad 1: /Input/I_LATCH_R -> Net-(U14-~{PL})
- U6 pad 10: Net-(U5-Q7) -> Net-(U14-Q7)
- U6 pad 11: Net-(BC16-NO) -> Net-(U6-D0)
- U6 pad 12: Net-(BC17-NO) -> Net-(U6-D1)
- U6 pad 13: Net-(BC18-NO) -> Net-(U6-D2)
- U6 pad 14: Net-(BC19-NO) -> Net-(U6-D3)
- U6 pad 15: Net-(U10-GND) -> GND
- U6 pad 2: /Input/I_CLK_R -> Net-(U14-CP)
- U6 pad 3: Net-(BC20-NO) -> Net-(U6-D4)
- U6 pad 8: Net-(U10-GND) -> GND
- U6 pad 9: Net-(U6-Q7) -> unconnected-(U6-Q7-Pad9)
- U7 pad 23: unconnected-(U7-GND-Pad23) -> GND
- U7 pad 3: unconnected-(U7-GND-Pad3) -> GND
- U7 pad 4: unconnected-(U7-GND-Pad4) -> GND
- U8 pad 1: /Input/I_LATCH_R -> Net-(U14-~{PL})
- U8 pad 10: Net-(U6-Q7) -> Net-(U5-Q7)
- U8 pad 11: Net-(U8-D0) -> Net-(BC3-NO)
- U8 pad 15: Net-(U10-GND) -> GND
- U8 pad 2: /Input/I_CLK_R -> Net-(U14-CP)
- U8 pad 3: Net-(U8-D4) -> Net-(E3-D)
- U8 pad 4: Net-(U8-D5) -> Net-(BC5-NO)
- U8 pad 5: Net-(U8-D6) -> Net-(BC4-NO)
- U8 pad 8: Net-(U10-GND) -> GND
- U8 pad 9: Net-(U10-DS) -> Net-(U14-DS)
- U9 pad 10: /Input/LED_BC6 -> /Input/LED_BC15
- U9 pad 11: /Input/LED_BC7 -> /Input/LED_BC12
- U9 pad 12: /Input/LED_BC8 -> /Input/LED_BC9
- U9 pad 13: /Input/LED_BC9 -> /Input/LED_BC7
- U9 pad 14: /Input/LED_BC10 -> unconnected-(U9-OUT9-Pad14)
- U9 pad 15: /Input/LED_BC11 -> unconnected-(U9-OUT10-Pad15)
- U9 pad 16: /Input/LED_BC12 -> /Input/LED_BC8
- U9 pad 17: /Input/LED_BC13 -> /Input/LED_BC17
- U9 pad 19: /Input/LED_BC15 -> /Input/LED_BC11
- U9 pad 20: /Input/LED_BC16 -> /Input/LED_BC10
- U9 pad 24: +5V -> +5VPW
- U9 pad 5: /Input/LED_BC1 -> /Input/LED_BC13
- U9 pad 6: /Input/LED_BC2 -> /Input/LED_BC16
- U9 pad 7: /Input/LED_BC3 -> /Input/LED_BC19
- U9 pad 8: /Input/LED_BC4 -> /Input/LED_BC20
- U9 pad 9: /Input/LED_BC5 -> /Input/LED_BC18
Routing:
- net +5V: track 0.00 -> 446.1 mm
- net /Input/LED_BC20: track 0.00 -> 228.2 mm
- net /Input/LED_BC17: track 0.00 -> 205.3 mm
- net /Input/LED_BC19: track 0.00 -> 201.2 mm
- net /Input/LED_BC18: track 0.00 -> 198.6 mm
- net /Input/LED_BC14: track 0.00 -> 176.8 mm
- net /Input/LED_BC15: track 0.00 -> 176.0 mm
- net /Input/LED_BC16: track 0.00 -> 176.0 mm
- net Net-(U14-CP): track 0.00 -> 169.7 mm
- net Net-(U14-~{PL}): track 0.00 -> 166.8 mm
- net /Input/LED_BC12: track 0.00 -> 153.5 mm
- net /Input/LED_BC13: track 0.00 -> 150.6 mm
- net /Input/LED_BC11: track 0.00 -> 148.8 mm
- net /Input/LED_BC1: track 0.00 -> 136.3 mm
- net /Input/LED_BC9: track 0.00 -> 130.0 mm
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- added copper zone on B.Cu, net GND
- added copper zone on F.Cu, net GND
Other:
- board size 363 x 166.2 mm -> 350.6 x 128.7 mm

Commit message: Nearly finished just need to add the footprint for the 5/6 pos switch and connect to the rest ! And it will be going into production !
Parts:
- added U3: ~, mf:7seg_x4, F.Cu at (118.5, 91.0)
- moved R33 9.82 mm to (259.9, 81.0), turned to 0 degrees
- moved C10 0.50 mm to (262.8, 99.2)
- moved U11 0.50 mm to (260.3, 85.9)
- turned E5 to 0 degrees
Connections:
- R33 pad 2: GND -> Net-(U11-ENB)
- U1 pad 10: /Input/I_CLK_R -> /Input/E5_B
- U1 pad 11: /Input/E5_B -> /Input/E4_B
- U1 pad 12: /Input/E5_A -> /Input/E4_A
- U1 pad 13: /Input/E4_B -> /Input/E2_B
- U1 pad 14: /Input/E4_A -> /Input/E1_B
- U1 pad 15: /Input/E3_B -> /Input/E1_A
- U1 pad 16: /Input/E3_A -> /Input/I_DATA_L
- U1 pad 17: /Input/E2_B -> /Input/I_LATCH_L
- U1 pad 18: /Input/E2_A -> /Input/I_CLK_L
- U1 pad 19: /Input/E1_B -> /Input/I_LATCH_R
- U1 pad 20: /Input/E1_A -> /Input/I_CLK_R
- U1 pad 5: /Input/I_CLK_L -> /Input/I_DATA_R
- U1 pad 6: /Input/I_DATA_L -> /Input/E2_A
- U1 pad 7: /Input/I_LATCH_L -> /Input/E3_B
- U1 pad 8: /Input/I_LATCH_R -> /Input/E3_A
- U1 pad 9: /Input/I_DATA_R -> /Input/E5_A
- U11 pad 2: Net-(U11-DAI) -> /Output/O_DATA
- U11 pad 21: GND -> Net-(U11-ENB)
- U11 pad 22: unconnected-(U11-DAO-Pad22) -> Net-(U11-DAO)
- U14 pad 1: Net-(U14-~{PL}) -> /Input/I_CLK_L
- U14 pad 2: Net-(U14-CP) -> /Input/I_LATCH_L
- U2 pad 3: /Output/O_8_DIN -> Net-(U2-DIN)
- U2 pad 4: /Output/O_8_CS -> Net-(U2-CS)
- U4 pad 3: Net-(U2-DOUT) -> /Output/O_8_DIN
- U4 pad 4: Net-(U2-LODA) -> /Output/O_8_CS
- U5 pad 1: Net-(U14-~{PL}) -> /Input/I_CLK_L
- U5 pad 10: unconnected-(U5-DS-Pad10) -> Net-(U5-DS)
- U5 pad 2: Net-(U14-CP) -> /Input/I_LATCH_L
- U5 pad 9: Net-(U5-Q7) -> /Input/I_DATA_L
- U6 pad 1: Net-(U14-~{PL}) -> /Input/I_CLK_L
- U6 pad 10: Net-(U14-Q7) -> unconnected-(U6-DS-Pad10)
- U6 pad 2: Net-(U14-CP) -> /Input/I_LATCH_L
- U6 pad 9: unconnected-(U6-Q7-Pad9) -> Net-(U14-DS)
- U7 pad 1: /Output/O_CLK -> unconnected-(U7-D1/TX-Pad1)
- U7 pad 13: /Output/O_8_DIN -> /Output/O_4_DIN
- U7 pad 14: /Output/O_8_CS -> /Output/O_4_CLK
- U7 pad 15: /Output/O_8_CLK -> /Output/O_DATA
- U7 pad 16: /Output/O_4_CLK -> /Output/O_CLK
- U7 pad 17: /Output/O_4_DIN -> /Output/O_LATCH
- U7 pad 18: unconnected-(U7-D19/A1-Pad18) -> /Output/O_8_CLK
- U7 pad 19: unconnected-(U7-D20/A2-Pad19) -> /Output/O_8_CS
- U7 pad 2: /Output/O_DATA -> unconnected-(U7-D0/RX-Pad2)
- U7 pad 20: unconnected-(U7-D21/A3-Pad20) -> /Output/O_8_DIN
- U7 pad 5: /Output/O_LATCH -> unconnected-(U7-D2-Pad5)
- U8 pad 1: Net-(U14-~{PL}) -> /Input/I_CLK_L
- U8 pad 10: Net-(U5-Q7) -> Net-(U14-Q7)
- U8 pad 2: Net-(U14-CP) -> /Input/I_LATCH_L
- U8 pad 9: Net-(U14-DS) -> Net-(U5-DS)
- U9 pad 10: /Input/LED_BC15 -> /Input/LED_BC19
- U9 pad 11: /Input/LED_BC12 -> /Input/LED_BC16
- U9 pad 12: /Input/LED_BC9 -> /Input/LED_BC13
- U9 pad 2: /Output/O_DATA -> Net-(U11-DAO)
- U9 pad 22: Net-(U11-DAI) -> unconnected-(U9-DAO-Pad22)
- U9 pad 5: /Input/LED_BC13 -> /Input/LED_BC9
- U9 pad 6: /Input/LED_BC16 -> /Input/LED_BC12
- U9 pad 7: /Input/LED_BC19 -> /Input/LED_BC15
- U9 pad 8: /Input/LED_BC20 -> /Input/LED_BC18
- U9 pad 9: /Input/LED_BC18 -> /Input/LED_BC20
Routing:
- net +5VPW: track 3.46 -> 1134.7 mm
- net /Input/I_CLK_R: track 0.00 -> 564.8 mm
- net /Input/I_LATCH_R: track 0.00 -> 506.9 mm
- net /Output/O_LATCH: track 0.00 -> 471.7 mm
- net Net-(U11-DAO): track 0.00 -> 467.3 mm
- net /Input/I_DATA_R: track 0.00 -> 467.3 mm
- net /Input/E5_A: track 0.00 -> 386.8 mm
- net /Input/E5_B: track 0.00 -> 381.9 mm
- net +5V: track 446.1 -> 782.5 mm
- net /Output/O_CLK: track 0.00 -> 306.8 mm
- net /Input/I_LATCH_L: track 0.00 -> 290.7 mm
- net /Input/I_CLK_L: track 0.00 -> 287.3 mm
- net /Output/O_4_CLK: track 0.00 -> 181.8 mm
- net /Output/O_4_DIN: track 0.00 -> 180.1 mm
- net Net-(U14-CP): track 169.7 -> 0.00 mm
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