File: mf.kicad_pcb (KiCad board)
At the start: 2 copper layers, 350.6 x 128.7 mm, 113 parts, among them U1 Sparkfun_Pro_Micro, U11 DM13a, U14 74HC165, U16 74HC165, U17 74HC165, U19 74HC165, U5 74HC165, U6 74HC165, U7 Sparkfun_Pro_Micro, U8 74HC165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

Commit message: last footprint and some graphics added
Parts:
- added U12: ~, mf:5_6-pos-switch, F.Cu at (159.5, 103.2)
- added U13: ~, mf:5_6-pos-switch, F.Cu at (159.5, 139.0)
Routing:
- net Net-(U16-D6): track 4.63 -> 68.7 mm
- net Net-(U16-D7): track 5.15 -> 67.1 mm
- net Net-(U16-D5): track 4.63 -> 64.1 mm
- net Net-(U16-D4): track 5.15 -> 60.0 mm
- net Net-(U16-D0): track 5.15 -> 47.2 mm
- net Net-(U6-D5): track 4.63 -> 43.1 mm
- net Net-(U16-D1): track 4.63 -> 42.6 mm
- net Net-(U16-D2): track 4.63 -> 41.0 mm
- net Net-(U6-D6): track 4.63 -> 39.1 mm
- net +5VPW: track 1134.7 -> 1167.7 mm
- net Net-(U6-D7): track 5.15 -> 37.2 mm
- net Net-(U16-D3): track 5.15 -> 31.2 mm
- net /Input/E4_B: track 165.5 -> 142.3 mm
- net /Input/E4_A: track 165.5 -> 146.7 mm
- net +5V: track 782.5 -> 796.9 mm
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Other:
- board text added: "Made by Gigi"

Commit message: Final commit (i hope) !
Connections:
- U17 pad 9: Net-(U17-Q7) -> Net-(U16-DS)
- U7 pad 13: /Output/O_4_DIN -> /Output/O_4_CLK
- U7 pad 14: /Output/O_4_CLK -> /Output/O_4_DIN
Routing:
- net Net-(U16-DS): track 0.00 -> 106.8 mm
- net +5VPW: track 1167.7 -> 1177.5 mm
- net /Input/E4_B: track 142.3 -> 150.6 mm
- net /Input/E4_A: track 146.7 -> 153.8 mm
- net Net-(U16-D2): track 41.0 -> 35.4 mm
- net /Output/O_4_DIN: track 180.7 -> 185.9 mm
- net /Input/I_CLK_R: track 564.8 -> 561.2 mm
- net Net-(U16-D1): track 42.6 -> 39.1 mm
- net Net-(U2-CS): track 61.6 -> 58.7 mm
- net Net-(U2-CLK-Pad5): track 66.9 -> 64.1 mm
- net Net-(BC5-NO): track 53.2 -> 51.3 mm
- net Net-(U2-DIN): track 55.1 -> 53.4 mm
- net /Input/E1_B: track 44.2 -> 42.5 mm
- net /Input/E3_B: track 123.3 -> 124.7 mm
- net /Input/E3_A: track 126.8 -> 128.2 mm
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