File: input.kicad_sch (KiCad schematic)
At the start: 113 parts, among them U10 74HC165, U14 74HC165, U16 74HC165, U17 74HC165, U19 74HC165, U5 74HC165, U6 74HC165, U8 74HC165

Commit message: Begin PCB routing + change in schematic
Parts:
- removed R59, R60, R61, R62, R63, R64, R65, R66, R67, R68, R69, R70, R71, R72, R73, R74, R75, R76, R77, R78, R79, R80, R81, R82: Resistor, Resistor_THT:R_Axial_DIN0207_L6.3mm_D2.5mm_P10.16mm_Horizontal, symbol PCM_SL_Devices:Resistor
- removed RB6: (no value), mf:r_but, symbol _mf:r_but
- removed U16, U19: 74HC165, Package_DIP:DIP-16_W7.62mm_LongPads, symbol 74xx:74HC165
- added R1, R17, R18, R19, R2, R20, R21, R22, R23, R24, R3, R34, R35, R36, R38, R39, R4, R40, R41, R42, R5, R6, R7, R8: Resistor, Resistor_THT:R_Axial_DIN0207_L6.3mm_D2.5mm_P10.16mm_Horizontal, symbol PCM_SL_Devices:Resistor
- added U21, U22: (no value), mf:3posswitch, symbol _mf:3_pos_switch
- added U5, U8: 74HC165, Package_DIP:DIP-16_W7.62mm_LongPads, symbol 74xx:74HC165
- renumbered R49 to R10, R48 to R11, R47 to R12, R46 to R13, R45 to R14, R44 to R15, R43 to R16, R42 to R25, R41 to R26, R40 to R27, R39 to R28, R38 to R29, R36 to R30, R35 to R31, R34 to R32, R32 to R43, R31 to R44, R30 to R45, R29 to R46, R28 to R47, R27 to R48, R26 to R49, R25 to R50, R24 to R59, R23 to R60, R22 to R61, R21 to R62, R20 to R63, R19 to R64, R18 to R65, R17 to R66, R50 to R9, U8 to U10, U6 to U16, U5 to U19, U10 to U6
Connections:
- net +5V: now also R59.2, R60.2, R61.2, R62.2, R1.1, R17.1, R18.1, R19.1, R2.1, R20.1, R21.1, R22.1, R23.1, R24.1, R3.1, R34.1, R35.1, R36.1, R38.1, R39.1, R4.1, R40.1, R41.1, R42.1, R5.1, R6.1, R7.1, R8.1, U5.16 (VCC), U8.16 (VCC); no longer R59.1, R60.1, R61.1, R62.1
- net GND: now also BC1.2 (C), BC10.2 (C), BC11.2 (C), BC12.2 (C), BC13.2 (C), BC14.2 (C), BC2.2 (C), BC3.2 (C), BC4.2 (C), BC5.2 (C), BC6.2 (C), BC7.2 (C), BC8.2 (C), BC9.2 (C), E5.2 (COM), E5.5 (E), RB5.2, U10.15 (~{CE}), U10.8 (GND), U14.15 (~{CE}), U14.8 (GND), U16.15 (~{CE}), U16.8 (GND), U17.15 (~{CE}), U17.8 (GND), U19.15 (~{CE}), U19.8 (GND), U6.15 (~{CE}), U6.8 (GND), U21.3 (GND), U22.3 (GND), U5.15 (~{CE}), U5.8 (GND), U8.15 (~{CE}), U8.8 (GND); no longer RB5.1
- net I_CLK_L: no longer U14.2 (CP), U17.2 (CP)
- net I_CLK_R: now also U17.2 (CP); no longer U6.2 (CP)
- net I_DATA_R: now also U19.9 (Q7); no longer U6.9 (Q7)
- net I_LATCH_L: no longer U14.1 (~{PL}), U17.1 (~{PL})
- net I_LATCH_R: now also U17.1 (~{PL}); no longer U6.1 (~{PL})
- net at U16.10 (DS): now also U10.9 (Q7); no longer U19.9 (Q7)
- net at R50.2, U16.11 (D0): now also U12. (GND); no longer BC16.3 (NO)
- net at R49.2, U16.12 (D1): now also U13. (GND); no longer BC17.3 (NO)
- net at R48.2, U16.13 (D2): now also U13. (GND); no longer BC18.3 (NO)
- net at R47.2, U16.14 (D3): now also U13. (GND); no longer BC19.3 (NO)
- net at R46.2, U16.3 (D4): now also U12. (GND); no longer BC20.3 (NO)
- net at R45.2, U16.4 (D5): now also U12. (GND)
- net at R44.2, U16.5 (D6): now also U12. (GND)
- net at R43.2, U16.6 (D7): now also U12. (GND)
- net at U16.9 (Q7): now also U19.10 (DS); no longer U10.10 (DS)
- net at R11.2, U6.4 (D5): now also U13. (GND)
- net at U14.9 (Q7): now also U6.10 (DS)
- net at BC1.3 (NO): now also R1.2, U5.11 (D0)
- net at BC2.3 (NO): now also R7.2, U5.5 (D6)
- net at BC3.3 (NO): now also R17.2, U8.11 (D0)
- net at BC4.3 (NO): now also R23.2, U8.5 (D6)
- net at BC5.3 (NO): now also R22.2, U8.4 (D5)
- net at BC6.3 (NO): now also U14.11 (D0), R34.2
- net at E5.4 (D): now also R53.2, U17.13 (D2)
- net at U15.1: now also R12.2, U6.3 (D4)
- net at U20.1: now also U14.6 (D7), R42.2
- net at R10.2, U6.5 (D6): now also U13. (GND)
- net at U17.4 (D5): now also BC15.3 (NO), R56.2; no longer U15.2
- net at R9.2, U6.6 (D7): now also U13. (GND)
- net at U17.5 (D6): now also BC12.3 (NO), R57.2; no longer U18.2
- net at U17.6 (D7): now also BC9.3 (NO), R58.2; no longer U18.1
- net at U17.11 (D0): now also R51.2; no longer U13. (GND)
- net at U17.12 (D1): now also BC8.3 (NO), R52.2; no longer U13. (GND)
- net at U17.14 (D3): now also BC7.3 (NO), R54.2; no longer U13. (GND)
- net at U17.3 (D4): now also BC18.3 (NO), R55.2; no longer U13. (GND)
- net at U17.9 (Q7): now also U10.10 (DS)
- net at R14.2, U6.13 (D2): now also U18.1
- net at U20.2: now also U14.14 (D3), R38.2
- net at U19.5 (D6): now also BC14.3 (NO), R65.2; no longer R60.2
- net at R15.2, U6.12 (D1): now also U18.2
- net at U14.10 (DS): now also U8.9 (Q7)
- net at R16.2, U6.11 (D0): now also U21.1
- net at R13.2, U6.14 (D3): now also U15.2
- new net: BC19.3 (NO), R62.1, U19.14 (D3)
- new net: R39.2, U14.3 (D4), U21.2
- new net: R41.2, U14.5 (D6), U22.2
- new net: R18.2, U8.12 (D1)
- new net: R20.2, U8.14 (D3)
- new net: BC11.3 (NO), R66.2, U19.6 (D7)
- new net: R35.2, RB4.2, U14.12 (D1)
- new net: E3.4 (D), R21.2, U8.3 (D4)
- new net: R6.2, U5.4 (D5)
- new net: R5.2, U5.3 (D4)
- new net: R24.2, RB5.1, U8.6 (D7)
- new net: E2.4 (D), R8.2, U5.6 (D7)
- new net: R4.2, U5.14 (D3)
- new net: BC13.3 (NO), R60.1, U19.12 (D1)
- new net: BC10.3 (NO), R59.1, U19.11 (D0)
- new net: BC16.3 (NO), R61.1, U19.13 (D2)
- new net: BC20.3 (NO), R63.2, U19.3 (D4)
- new net: BC17.3 (NO), R64.2, U19.4 (D5)
- new net: U14.1 (~{PL}), U5.1 (~{PL}), U6.1 (~{PL}), U8.1 (~{PL})
- new net: U5.9 (Q7), U8.10 (DS)
- new net: R19.2, U8.13 (D2)
- new net: U14.2 (CP), U5.2 (CP), U6.2 (CP), U8.2 (CP)
- new net: R3.2, U5.13 (D2)
- new net: R40.2, U14.4 (D5), U22.1
- new net: E4.4 (D), R36.2, U14.13 (D2)
- new net: E1.4 (D), R2.2, U5.12 (D1)
- no-connect marks 30 -> 35
Other:
- moved on the sheet: BC1, BC10, BC11, BC12, BC13, BC14, BC15, BC16, BC17, BC18, BC19, BC2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

Commit message: Nearly finished just need to add the footprint for the 5/6 pos switch and connect to the rest ! And it will be going into production !
Connections:
- net I_CLK_L: now also U14.1 (~{PL}), U5.1 (~{PL}), U6.1 (~{PL}), U8.1 (~{PL})
- net I_DATA_L: now also U5.9 (Q7)
- net I_LATCH_L: now also U14.2 (CP), U5.2 (CP), U6.2 (CP), U8.2 (CP)
- net at U8.10 (DS): now also U14.9 (Q7); no longer U5.9 (Q7)
- net at U8.9 (Q7): now also U5.10 (DS); no longer U14.10 (DS)
- net at U6.10 (DS): no longer U14.9 (Q7)
- net at U6.9 (Q7): now also U14.10 (DS)
- no-connect marks 35 -> 26

Commit message: last footprint and some graphics added
Parts:
- U12, U13: footprint (none) -> mf:5_6-pos-switch
Connections:
- net GND: now also U12.7 (GND), U13.7 (GND); no longer U12. (GND), U13. (GND)
- net at R50.2, U16.11 (D0): now also U12.4; no longer U12. (GND)
- net at R49.2, U16.12 (D1): now also U12.3; no longer U13. (GND)
- net at R48.2, U16.13 (D2): now also U12.2; no longer U13. (GND)
- net at R47.2, U16.14 (D3): now also U12.1; no longer U13. (GND)
- net at R46.2, U16.3 (D4): now also U13.1; no longer U12. (GND)
- net at R45.2, U16.4 (D5): now also U13.2; no longer U12. (GND)
- net at R44.2, U16.5 (D6): now also U13.3; no longer U12. (GND)
- net at R43.2, U16.6 (D7): now also U12.5; no longer U12. (GND)
- net at R11.2, U6.4 (D5): now also U13.4; no longer U13. (GND)
- net at R10.2, U6.5 (D6): now also U13.5; no longer U13. (GND)
- net at R9.2, U6.6 (D7): now also U13.6; no longer U13. (GND)

Commit message: Final commit (i hope) !
Parts:
- removed C4: Capacitor_NP, Capacitor_THT:C_Disc_D3.0mm_W2.0mm_P2.50mm, symbol PCM_SL_Devices:Capacitor_NP
- removed R25, R26, R27, R28, R29, R30, R31, R32: Resistor, Resistor_THT:R_Axial_DIN0207_L6.3mm_D2.5mm_P10.16mm_Horizontal, symbol PCM_SL_Devices:Resistor
- removed U10: 74HC165, Package_DIP:DIP-16_W7.62mm_LongPads, symbol 74xx:74HC165
Connections:
- net at U16.10 (DS): now also U17.9 (Q7)
- no-connect marks 26 -> 25
